File: mcu.kicad_sch (KiCad schematic)
At the start: 23 parts, among them J6 Conn_01x08, J7 Conn_01x02, U5 AT25XE321D-UUN-T, U6 EFM32PG23B200F512IM40, Y2 39MHz

Commit message: G2 revision
G2 revision = Kampela development kit

Features:
- electronics is more stable and reliable
- better power harvesting efficiency
- fixed a touchscreen instability with powerful NFC transmitters
- mechanical layout improved for low-volume productions for a devkit batch
- NFC coil placed closer to the phone antenna. The coil parameters are optimized based on a mathematical model of the NFS harvester circuit.
Parts:
- J6: footprint MyLib:PinHeader_1x08_P1.27mm_Vertical_Prog -> MyLib:PinHeader_1x08_P1.27mm_Vertical
- R?: now not fitted

Commit message: G5 revision
Parts:
- removed TP?: TestPoint, TestPoint:TestPoint_Pad_D1.0mm, symbol Connector:TestPoint
- added TP? (x5): TestPoint, TestPoint:TestPoint_Pad_D1.0mm, symbol Connector:TestPoint
- C?: value 1x50 -> 1x6.3
- C?: value 4.7x25 -> 1x6.3
Connections:
- net P_GOOD: now also TP?.1
- net RX: now also TP?.1
- net SWDCK: now also TP?.1
- net SWDIO: now also TP?.1
- net TX: now also TP?.1
