File: mcuSec.kicad_sch (KiCad schematic)
At the start: 27 parts, among them J6 Conn_01x08, J7 Conn_01x02, U5 AT25XE321D-UUN-T, U6 EFM32PG23B200F512IM40, Y2 39MHz

Commit message: Next revision
Parts:
- removed C? (x7): 0.1u, Capacitor_SMD:C_0402_1005Metric, symbol Device:C
- removed C? (x2): 1x6.3, Capacitor_SMD:C_0402_1005Metric, symbol Device:C
- removed FB?: BLM15AG102SZ1D, Inductor_SMD:L_0402_1005Metric, symbol Device:FerriteBead_Small
- removed J7: Conn_01x02, Connector_PinHeader_1.27mm:PinHeader_1x02_P1.27mm_Vertical, symbol Connector_Generic:Conn_01x02
- removed R?: 2.2, Resistor_SMD:R_0603_1608Metric, symbol Device:R
- removed R? (x2): 10K, Resistor_SMD:R_0402_1005Metric, symbol Device:R
- removed R?: 1K, Resistor_SMD:R_0402_1005Metric, symbol Device:R
- removed Y?: FC2012AN, MyLib:Crystal_SMD_2012-2Pin_2.0x1.2mm, symbol Device:Crystal_Small
- added C39, C40, C42, C43, C44, C46: 0.1, Capacitor_SMD:C_0201_0603Metric, symbol Device:C
- added C41, C45: 1x6.3, Capacitor_SMD:C_0402_1005Metric, symbol Device:C
- added R16: 2.2, Resistor_SMD:R_0603_1608Metric, symbol Device:R
- added R17, R18: 10K, Resistor_SMD:R_0201_0603Metric, symbol Device:R
- renumbered J6 to J4, U5 to U6, U6 to U7, Y2 to Y1
Connections:
- net +1V8: now also U7.35 (AVDD), C39.2, C40.2, C41.1, C42.2, C43.2, C44.2, R18.2
- net GND: now also C39.1, C40.1, C41.2, C42.1, C43.1, C44.1, C45.2, C46.1, R17.1
- net P_GOOD: now also C46.2, R18.1
- net P_IN: now also R16.1
- net at D?.2 (A): now also R16.2, R17.2
- net GIMEL: now reaches U7.16 (PB03)
- net BET: now reaches U7.17 (PB02)
- net ALEPH: now reaches U7.19 (PB00)
- net at U7.30 (CAP): now also C45.1
- net EXTIN: now reaches U7.39 (PD01)
- net D_CS: now reaches U7.40 (PD00)
- net 2V8_EN renamed HET
- net BUSY renamed DALET
- net CS renamed TET
- net D/C renamed YOD
- net RES renamed VAV
- net RES_TC renamed ZAYIN
- net SCK renamed E_SCK
- net SDI renamed E_MOSI
- net ~{MCU_OK} renamed HE
Other:
- moved on the sheet: D?
